Commit message: change color of wheels to green

File: p_fpower_description/urdf/p_fpower.gazebo.xacro (robot description, xacro)
@@ -15,5 +15,5 @@
     <maxVel>0.1</maxVel>
     <fdir1>1 0 0</fdir1>
-    <material>Gazebo/FlatBlack</material>
+    <material>Gazebo/Green</material>
   </gazebo>
   <gazebo reference="wheel_right_link">
@@ -25,5 +25,5 @@
     <maxVel>0.1</maxVel>
     <fdir1>1 0 0</fdir1>
-    <material>Gazebo/FlatBlack</material>
+    <material>Gazebo/Green</material>
   </gazebo>
   <gazebo reference="caster_back_right_link">
@@ -34,5 +34,5 @@
     <minDepth>0.001</minDepth>
     <maxVel>1.0</maxVel>
-    <material>Gazebo/FlatBlack</material>
+    <material>Gazebo/Green</material>
   </gazebo>
   <gazebo reference="caster_back_left_link">
@@ -43,5 +43,5 @@
     <minDepth>0.001</minDepth>
     <maxVel>1.0</maxVel>
-    <material>Gazebo/FlatBlack</material>
+    <material>Gazebo/Green</material>
   </gazebo>
   <gazebo reference="imu_link">
@@ -103,5 +103,5 @@
   </gazebo>
   <gazebo reference="base_scan">
-    <material>Gazebo/FlatBlack</material>
+    <material>Gazebo/Green</material>
     <sensor type="ray" name="lds_lfcd_sensor">
       <pose>0 0 0 0 0 0</pose>

File: p_fpower_description/urdf/p_fpower.urdf.xacro (robot description, xacro)
@@ -43,5 +43,5 @@
         <mesh filename="package://turtlebot3_description/meshes/wheels/left_tire.stl" scale="0.001 0.001 0.001"/>
       </geometry>
-      <material name="dark"/>
+      <material name="green"/>
     </visual>
     <collision>
@@ -71,5 +71,5 @@
         <mesh filename="package://turtlebot3_description/meshes/wheels/right_tire.stl" scale="0.001 0.001 0.001"/>
       </geometry>
-      <material name="dark"/>
+      <material name="green"/>
     </visual>
     <collision>
@@ -144,5 +144,5 @@
         <mesh filename="package://turtlebot3_description/meshes/sensors/lds.stl" scale="0.001 0.001 0.001"/>
       </geometry>
-      <material name="dark"/>
+      <material name="green"/>
     </visual>
     <collision>

Commit message: add xacro macros and diff_drive

File: p_fpower_description/urdf/p_fpower.gazebo.xacro (robot description, xacro)
@@ -1,7 +1,8 @@
 <?xml version="1.0"?>
-<robot name="turtlebot3_waffle_pi_sim" xmlns:xacro="http://ros.org/wiki/xacro">
+<robot name="p_fpower_sim" xmlns:xacro="http://ros.org/wiki/xacro">
   <xacro:arg name="laser_visual"  default="false"/>
   <xacro:arg name="camera_visual" default="false"/>
   <xacro:arg name="imu_visual"    default="false"/>
+  <xacro:include filename="$(find $p_fpower_description)/urdf/ros_diff_drive.gazebo.xacro"/>
   <gazebo reference="base_link">
     <material>Gazebo/DarkGrey</material>
@@ -52,5 +53,5 @@
     <material>Gazebo/Grey</material>
   </gazebo>
-  <gazebo>
+  <!-- <gazebo>
     <plugin name="turtlebot3_waffle_pi_controller" filename="libgazebo_ros_diff_drive.so">
       <commandTopic>cmd_vel</commandTopic>
@@ -73,5 +74,5 @@
       <rosDebugLevel>na</rosDebugLevel>
     </plugin>
-  </gazebo>
+  </gazebo> -->
   <gazebo>
     <plugin name="imu_plugin" filename="libgazebo_ros_imu.so">

File: p_fpower_description/urdf/p_fpower.urdf.xacro (robot description, xacro)
@@ -1,6 +1,19 @@
 <?xml version="1.0" ?>
-<robot name="turtlebot3_waffle_pi" xmlns:xacro="http://ros.org/wiki/xacro">
-  <xacro:include filename="$(find p_fpower_description)/urdf/common_properties.xacro"/>
-  <xacro:include filename="$(find p_fpower_description)/urdf/p_fpower.gazebo.xacro"/>
+<robot name="p_moliveira" xmlns:xacro="http://ros.org/wiki/xacro">
+  <!--  Xacro description of turtlebot robot waffle pi used to play team hunt.-->
+  <!--  Francisco Power-->
+  <!--  PARI, November 2020-->
+  <!--Args are local, properties are global, so we copy the values of the arguments to the properties-->
+  <xacro:arg name="player_name" default="p_fpower" />
+  <xacro:arg name="player_color" default="Green" /> <!-- e.g. Red, Orange. Must exist in Gazebo/Colors and be defined in properties.xacro.-->
+  <!--Properties are global so they can be viewed from inside the included xacros-->
+  <!--  args are used with $(arg arg_name), properties are used as ${property_name}-->
+  <xacro:property name="player_name" value="$(arg player_name)"/>
+  <xacro:property name="player_color" value="$(arg player_color)"/>
+  <!-- Include other files-->
+  <xacro:include filename="$(find ${player_name}_description)/urdf/properties.xacro"/>
+  <!--  <xacro:include filename="$(find ${player_name}_description)/urdf/player.gazebo.xacro"/>-->
+  <xacro:include filename="$(find ${player_name}_description)/urdf/p_fpower.gazebo.macro.xacro"/>
+  <xacro:gazebo_macro player_color="Orange" laser_visual="true" camera_visual="false" imu_visual="true"/>
   <link name="base_footprint"/>
   <joint name="base_joint" type="fixed">

File: p_fpower_description/urdf/properties.xacro (robot description, xacro)
@@ -2,8 +2,8 @@
 <robot name="xacro_properties" xmlns:xacro="http://ros.org/wiki/xacro">
   <!-- Init colour -->
-  <material name="black">
+  <material name="Black">
       <color rgba="0.0 0.0 0.0 1.0"/>
   </material>
-  <material name="dark">
+  <material name="Dark">
     <color rgba="0.3 0.3 0.3 1.0"/>
   </material>
@@ -11,23 +11,23 @@
     <color rgba="0.4 0.4 0.4 1.0"/>
   </material>
-  <material name="blue">
+  <material name="Blue">
     <color rgba="0.0 0.0 0.8 1.0"/>
   </material>
-  <material name="green">
+  <material name="Green">
     <color rgba="0.0 0.8 0.0 1.0"/>
   </material>
-  <material name="grey">
+  <material name="Grey">
     <color rgba="0.5 0.5 0.5 1.0"/>
   </material>
-  <material name="orange">
+  <material name="Orange">
     <color rgba="${255/255} ${108/255} ${10/255} 1.0"/>
   </material>
-  <material name="brown">
+  <material name="Brown">
     <color rgba="${222/255} ${207/255} ${195/255} 1.0"/>
   </material>
-  <material name="red">
+  <material name="Red">
     <color rgba="0.8 0.0 0.0 1.0"/>
   </material>
-  <material name="white">
+  <material name="White">
     <color rgba="1.0 1.0 1.0 1.0"/>
   </material>

Commit message: telop basic control working

File: p_fpower_description/urdf/p_fpower.gazebo.xacro (robot description, xacro)
@@ -4,5 +4,5 @@
   <xacro:arg name="camera_visual" default="false"/>
   <xacro:arg name="imu_visual"    default="false"/>
-  <xacro:include filename="$(find p_fpower_description)/urdf/ros_diff_drive.gazebo.xacro"/>
+  <!-- <xacro:include filename="$(find p_fpower_description)/urdf/ros_diff_drive.gazebo.xacro"/> -->
   <gazebo reference="base_link">
     <material>Gazebo/DarkGrey</material>
@@ -53,5 +53,5 @@
     <material>Gazebo/Grey</material>
   </gazebo>
-  <!-- <gazebo>
+  <gazebo>
     <plugin name="turtlebot3_waffle_pi_controller" filename="libgazebo_ros_diff_drive.so">
       <commandTopic>cmd_vel</commandTopic>
@@ -74,5 +74,5 @@
       <rosDebugLevel>na</rosDebugLevel>
     </plugin>
-  </gazebo> -->
+  </gazebo>
   <gazebo>
     <plugin name="imu_plugin" filename="libgazebo_ros_imu.so">

File: p_fpower_description/urdf/p_fpower.urdf.xacro (robot description, xacro)
@@ -56,5 +56,5 @@
         <mesh filename="package://turtlebot3_description/meshes/wheels/left_tire.stl" scale="0.001 0.001 0.001"/>
       </geometry>
-      <material name="green"/>
+      <material name="Green"/>
     </visual>
     <collision>
@@ -84,5 +84,5 @@
         <mesh filename="package://turtlebot3_description/meshes/wheels/right_tire.stl" scale="0.001 0.001 0.001"/>
       </geometry>
-      <material name="green"/>
+      <material name="Green"/>
     </visual>
     <collision>
@@ -157,5 +157,5 @@
         <mesh filename="package://turtlebot3_description/meshes/sensors/lds.stl" scale="0.001 0.001 0.001"/>
       </geometry>
-      <material name="green"/>
+      <material name="Green"/>
     </visual>
     <collision>

File: p_fpower_description/urdf/ros_diff_drive.gazebo.xacro (robot description, xacro)
@@ -5,5 +5,5 @@
         <odometryFrame>odom</odometryFrame>
         <odometrySource>world</odometrySource>
-        <publishOdomTF>false</publishOdomTF>
+        <publishOdomTF>true</publishOdomTF>
         <!--      <publishOdomTF>true</publishOdomTF>-->
         <robotBaseFrame>base_footprint</robotBaseFrame>

Commit message: color, player name properties, separate controller

File: p_fpower_description/urdf/p_fpower.gazebo.xacro (robot description, xacro)
@@ -4,5 +4,13 @@
   <xacro:arg name="camera_visual" default="false"/>
   <xacro:arg name="imu_visual"    default="false"/>
-  <!-- <xacro:include filename="$(find p_fpower_description)/urdf/ros_diff_drive.gazebo.xacro"/> -->
+  <!--Args are local, properties are global, so we copy the values of the arguments to the properties-->
+  <xacro:arg name="player_name" default="p_fpower" />
+  <xacro:arg name="player_color" default="Green" /> <!-- e.g. Red, Orange. Must exist in Gazebo/Colors and be defined in properties.xacro.-->
+  <!--Properties are global so they can be viewed from inside the included xacros-->
+  <!--  args are used with $(arg arg_name), properties are used as ${property_name}-->
+  <xacro:property name="player_name" value="$(arg player_name)"/>
+  <xacro:property name="player_color" value="$(arg player_color)"/>
+  <!-- include controller file -->
+  <xacro:include filename="$(find ${player_name}_description)/urdf/ros_diff_drive.gazebo.xacro"/>
   <gazebo reference="base_link">
     <material>Gazebo/DarkGrey</material>
@@ -16,5 +24,5 @@
     <maxVel>0.1</maxVel>
     <fdir1>1 0 0</fdir1>
-    <material>Gazebo/Green</material>
+    <material>Gazebo/${player_color}</material>
   </gazebo>
   <gazebo reference="wheel_right_link">
@@ -26,5 +34,5 @@
     <maxVel>0.1</maxVel>
     <fdir1>1 0 0</fdir1>
-    <material>Gazebo/Green</material>
+    <material>Gazebo/${player_color}</material>
   </gazebo>
   <gazebo reference="caster_back_right_link">
@@ -35,5 +43,5 @@
     <minDepth>0.001</minDepth>
     <maxVel>1.0</maxVel>
-    <material>Gazebo/Green</material>
+    <material>Gazebo/${player_color}</material>
   </gazebo>
   <gazebo reference="caster_back_left_link">
@@ -44,5 +52,5 @@
     <minDepth>0.001</minDepth>
     <maxVel>1.0</maxVel>
-    <material>Gazebo/Green</material>
+    <material>Gazebo/${player_color}</material>
   </gazebo>
   <gazebo reference="imu_link">
@@ -52,26 +60,4 @@
     </sensor>
     <material>Gazebo/Grey</material>
-  </gazebo>
-  <gazebo>
-    <plugin name="turtlebot3_waffle_pi_controller" filename="libgazebo_ros_diff_drive.so">
-      <commandTopic>cmd_vel</commandTopic>
-      <odometryTopic>odom</odometryTopic>
-      <odometryFrame>odom</odometryFrame>
-      <odometrySource>world</odometrySource>
-      <publishOdomTF>true</publishOdomTF>
-      <robotBaseFrame>base_footprint</robotBaseFrame>
-      <publishWheelTF>false</publishWheelTF>
-      <publishTf>true</publishTf>
-      <publishWheelJointState>true</publishWheelJointState>
-      <legacyMode>false</legacyMode>
-      <updateRate>30</updateRate>
-      <leftJoint>wheel_left_joint</leftJoint>
-      <rightJoint>wheel_right_joint</rightJoint>
-      <wheelSeparation>0.287</wheelSeparation>
-      <wheelDiameter>0.066</wheelDiameter>
-      <wheelAcceleration>1</wheelAcceleration>
-      <wheelTorque>10</wheelTorque>
-      <rosDebugLevel>na</rosDebugLevel>
-    </plugin>
   </gazebo>
   <gazebo>
@@ -104,5 +90,5 @@
   </gazebo>
   <gazebo reference="base_scan">
-    <material>Gazebo/Green</material>
+    <material>Gazebo/${player_color}</material>
     <sensor type="ray" name="lds_lfcd_sensor">
       <pose>0 0 0 0 0 0</pose>

File: p_fpower_description/urdf/p_fpower.urdf.xacro (robot description, xacro)
@@ -56,5 +56,5 @@
         <mesh filename="package://turtlebot3_description/meshes/wheels/left_tire.stl" scale="0.001 0.001 0.001"/>
       </geometry>
-      <material name="Green"/>
+      <material name="${player_color}"/>
     </visual>
     <collision>
@@ -84,5 +84,5 @@
         <mesh filename="package://turtlebot3_description/meshes/wheels/right_tire.stl" scale="0.001 0.001 0.001"/>
       </geometry>
-      <material name="Green"/>
+      <material name="${player_color}"/>
     </visual>
     <collision>
@@ -157,5 +157,5 @@
         <mesh filename="package://turtlebot3_description/meshes/sensors/lds.stl" scale="0.001 0.001 0.001"/>
       </geometry>
-      <material name="Green"/>
+      <material name="${player_color}"/>
     </visual>
     <collision>

File: p_fpower_description/urdf/ros_diff_drive.gazebo.xacro (robot description, xacro)
@@ -1,31 +1,33 @@
-<gazebo>
-    <plugin name="turtlebot3_waffle_pi_controller" filename="libgazebo_ros_diff_drive.so">
-        <commandTopic>cmd_vel</commandTopic>
-        <odometryTopic>odom</odometryTopic>
-        <odometryFrame>odom</odometryFrame>
-        <odometrySource>world</odometrySource>
-        <publishOdomTF>true</publishOdomTF>
-        <!--      <publishOdomTF>true</publishOdomTF>-->
-        <robotBaseFrame>base_footprint</robotBaseFrame>
-        <publishWheelTF>false</publishWheelTF>
-        <publishTf>true</publishTf>
-        <publishWheelJointState>true</publishWheelJointState>
-        <legacyMode>false</legacyMode>
-        <updateRate>30</updateRate>
-        <leftJoint>wheel_left_joint</leftJoint>
-        <rightJoint>wheel_right_joint</rightJoint>
-        <wheelSeparation>0.287</wheelSeparation>
-        <wheelDiameter>0.066</wheelDiameter>
-        <wheelAcceleration>1</wheelAcceleration>
-        <wheelTorque>10</wheelTorque>
-        <rosDebugLevel>na</rosDebugLevel>
-        <linear>
-            <x>
-                <has_velocity_limits>true</has_velocity_limits>
-                <max_velocity>0.1</max_velocity>
-                <min_velocity>-0.1</min_velocity>
-            </x>
-        </linear>
-        <publish_cmd>truesads</publish_cmd>
-    </plugin>
-</gazebo>
+<?xml version="1.0"?>
+<robot name="p_fpower_ros_diff_drive" xmlns:xacro="http://ros.org/wiki/xacro">
+    <gazebo>
+        <plugin name="turtlebot3_waffle_pi_controller" filename="libgazebo_ros_diff_drive.so">
+            <commandTopic>cmd_vel</commandTopic>
+            <odometryTopic>odom</odometryTopic>
+            <odometryFrame>odom</odometryFrame>
+            <odometrySource>world</odometrySource>
+            <publishOdomTF>true</publishOdomTF>
+            <robotBaseFrame>base_footprint</robotBaseFrame>
+            <publishWheelTF>false</publishWheelTF>
+            <publishTf>true</publishTf>
+            <publishWheelJointState>true</publishWheelJointState>
+            <legacyMode>false</legacyMode>
+            <updateRate>30</updateRate>
+            <leftJoint>wheel_left_joint</leftJoint>
+            <rightJoint>wheel_right_joint</rightJoint>
+            <wheelSeparation>0.287</wheelSeparation>
+            <wheelDiameter>0.066</wheelDiameter>
+            <wheelAcceleration>1</wheelAcceleration>
+            <wheelTorque>10</wheelTorque>
+            <rosDebugLevel>na</rosDebugLevel>
+            <linear>
+                <x>
+                    <has_velocity_limits>true</has_velocity_limits>
+                    <max_velocity>0.1</max_velocity>
+                    <min_velocity>-0.1</min_velocity>
+                </x>
+            </linear>
+            <publish_cmd>truesads</publish_cmd>
+        </plugin>
+    </gazebo>
+</robot>
