Commit message: new controller

File: p_fpower_description/urdf/p_fpower.urdf.xacro (robot description, xacro)
@@ -8,12 +8,11 @@
   <xacro:arg name="player_color" default="Green" /> <!-- e.g. Red, Orange. Must exist in Gazebo/Colors and be defined in properties.xacro.-->
   <!--Properties are global so they can be viewed from inside the included xacros-->
-  <!--  args are used with $(arg arg_name), properties are used as ${property_name}-->
   <xacro:property name="player_name" value="$(arg player_name)"/>
   <xacro:property name="player_color" value="$(arg player_color)"/>
   <!-- Include other files-->
   <xacro:include filename="$(find ${player_name}_description)/urdf/properties.xacro"/>
-   <xacro:include filename="$(find ${player_name}_description)/urdf/p_fpower.gazebo.xacro"/>
-  <!-- <xacro:include filename="$(find ${player_name}_description)/urdf/p_fpower.gazebo.macro.xacro"/>
-  <xacro:gazebo_macro player_color="Orange" laser_visual="true" camera_visual="false" imu_visual="true"/> -->
+   <!-- <xacro:include filename="$(find ${player_name}_description)/urdf/p_fpower.gazebo.xacro"/> -->
+  <xacro:include filename="$(find ${player_name}_description)/urdf/p_fpower.gazebo.macro.xacro"/>
+  <xacro:gazebo_macro player_name="${player_name}" player_color="${player_color}" laser_visual="false" camera_visual="false" imu_visual="false"/>
   <link name="base_footprint"/>
   <joint name="base_joint" type="fixed">

File: p_fpower_description/urdf/ros_control.gazebo.xacro (robot description, xacro)
@@ -1,24 +1,27 @@
-<!--  Launch the library plygin for the ROS native controller -->
-<gazebo>
-    <plugin name="gazebo_ros_control" filename="libgazebo_ros_control.so"></plugin>
-</gazebo>
-<transmission name="left_wheel_transmission">
-    <type>transmission_interface/SimpleTransmission</type>
-    <joint name="wheel_left_joint" >
-        <hardwareInterface>hardware_interface/VelocityJointInterface</hardwareInterface>
-    </joint>
-    <actuator name="left_wheel_actuator" >
-        <mechanicalReduction>7</mechanicalReduction>
-        <hardwareInterface>VelocityJointInterface</hardwareInterface>
-    </actuator>
-</transmission>
-<transmission name="right_wheel_transmission">
-    <type>transmission_interface/SimpleTransmission</type>
-    <joint name="wheel_right_joint">
-        <hardwareInterface>hardware_interface/VelocityJointInterface</hardwareInterface>
-    </joint>
-    <actuator name="right_wheel_actuator">
-        <mechanicalReduction>7</mechanicalReduction>
-        <hardwareInterface>VelocityJointInterface</hardwareInterface>
-    </actuator>
-</transmission>
+<?xml version="1.0"?>
+<robot name="p_fpower_ros_control" xmlns:xacro="http://ros.org/wiki/xacro">
+    <!--  Launch the library plygin for the ROS native controller -->
+    <gazebo>
+        <plugin name="gazebo_ros_control" filename="libgazebo_ros_control.so"></plugin>
+    </gazebo>
+    <transmission name="left_wheel_transmission">
+        <type>transmission_interface/SimpleTransmission</type>
+        <joint name="wheel_left_joint">
+            <hardwareInterface>hardware_interface/VelocityJointInterface</hardwareInterface>
+        </joint>
+        <actuator name="left_wheel_actuator">
+            <mechanicalReduction>7</mechanicalReduction>
+            <hardwareInterface>VelocityJointInterface</hardwareInterface>
+        </actuator>
+    </transmission>
+    <transmission name="right_wheel_transmission">
+        <type>transmission_interface/SimpleTransmission</type>
+        <joint name="wheel_right_joint">
+            <hardwareInterface>hardware_interface/VelocityJointInterface</hardwareInterface>
+        </joint>
+        <actuator name="right_wheel_actuator">
+            <mechanicalReduction>7</mechanicalReduction>
+            <hardwareInterface>VelocityJointInterface</hardwareInterface>
+        </actuator>
+    </transmission>
+</robot>
