Commit message: player color arguent added

File: p_fpower_description/urdf/p_fpower.gazebo.macro.xacro (robot description, xacro)
@@ -1,8 +1,8 @@
 <?xml version="1.0"?>
 <robot name="p_fpower_sim" xmlns:xacro="http://ros.org/wiki/xacro">
-  <xacro:macro name="gazebo_macro" params="player_name player_color laser_visual camera_visual imu_visual" >
+  <xacro:macro name="gazebo_macro" params="player_color laser_visual camera_visual imu_visual" >
     <!-- include controller file -->
-    <!-- <xacro:include filename="$(find ${player_name}_description)/urdf/ros_diff_drive.gazebo.xacro" /> -->
-    <xacro:include filename="$(find ${player_name}_description)/urdf/ros_control.gazebo.xacro" />
+    <!-- <xacro:include filename="$(find p_fpower_description)/urdf/ros_diff_drive.gazebo.xacro" /> -->
+    <xacro:include filename="$(find p_fpower_description)/urdf/ros_control.gazebo.xacro" />
     <gazebo reference="base_link">
       <material>Gazebo/DarkGrey</material>

File: p_fpower_description/urdf/p_fpower.urdf.xacro (robot description, xacro)
@@ -5,14 +5,12 @@
   <!--  PARI, November 2020-->
   <!--Args are local, properties are global, so we copy the values of the arguments to the properties-->
-  <xacro:arg name="player_name" default="p_fpower" />
   <xacro:arg name="player_color" default="Green" /> <!-- e.g. Red, Orange. Must exist in Gazebo/Colors and be defined in properties.xacro.-->
   <!--Properties are global so they can be viewed from inside the included xacros-->
-  <xacro:property name="player_name" value="$(arg player_name)"/>
   <xacro:property name="player_color" value="$(arg player_color)"/>
   <!-- Include other files-->
-  <xacro:include filename="$(find ${player_name}_description)/urdf/properties.xacro"/>
-   <!-- <xacro:include filename="$(find ${player_name}_description)/urdf/p_fpower.gazebo.xacro"/> -->
-  <xacro:include filename="$(find ${player_name}_description)/urdf/p_fpower.gazebo.macro.xacro"/>
-  <xacro:gazebo_macro player_name="${player_name}" player_color="${player_color}" laser_visual="false" camera_visual="false" imu_visual="false"/>
+  <xacro:include filename="$(find p_fpower_description)/urdf/properties.xacro"/>
+   <!-- <xacro:include filename="$(find p_fpower_description)/urdf/p_fpower.gazebo.xacro"/> -->
+  <xacro:include filename="$(find p_fpower_description)/urdf/p_fpower.gazebo.macro.xacro"/>
+  <xacro:gazebo_macro player_color="${player_color}" laser_visual="false" camera_visual="false" imu_visual="false"/>
   <link name="base_footprint"/>
   <joint name="base_joint" type="fixed">

Commit message: colision created, not being detected

File: p_fpower_description/urdf/p_fpower.gazebo.macro.xacro (robot description, xacro)
@@ -120,5 +120,4 @@
         <camera>
           <horizontal_fov>1.085595</horizontal_fov>
-          <!-- <horizontal_fov>2.899921</horizontal_fov> -->
           <image>
             <!-- <width>640</width> -->
@@ -148,4 +147,18 @@
       </sensor>
     </gazebo>
+    <gazebo reference="base_link">
+      <sensor name="base_link" type="contact">
+        <update_rate>1000.0</update_rate>
+        <always_on>true</always_on>
+        <contact>
+          <collision>base_footprint_fixed_joint_lump__base_link_collision_collision</collision>
+        </contact>
+        <plugin name="base_link_contact_sensor_plugin" filename="libgazebo_ros_bumper.so">
+          <bumperTopicName>contact</bumperTopicName>
+          <!-- <frameName>world</frameName> -->
+          <frameName>base_footprint</frameName>
+        </plugin>
+      </sensor>
+    </gazebo>
   </xacro:macro>
 </robot>

Commit message: contact detection working

File: p_fpower_description/urdf/p_fpower.gazebo.macro.xacro (robot description, xacro)
@@ -152,10 +152,9 @@
         <always_on>true</always_on>
         <contact>
-          <collision>base_footprint_fixed_joint_lump__base_link_collision_collision</collision>
+          <collision>base_footprint_fixed_joint_lump__base_link_collision</collision>
         </contact>
         <plugin name="base_link_contact_sensor_plugin" filename="libgazebo_ros_bumper.so">
           <bumperTopicName>contact</bumperTopicName>
-          <!-- <frameName>world</frameName> -->
-          <frameName>base_footprint</frameName>
+          <frameName>world</frameName>
         </plugin>
       </sensor>
